File: Opto_8/rtn_sub_4x.kicad_sch (KiCad schematic)
At the start: 23 parts, among them U6 LM339

Commit message: in16_drv8
Parts:
- removed C35, C36, C38, C39: 100n, Capacitor_SMD:C_0402_1005Metric, symbol Device:C
- removed D10, D7, D8, D9: 1N4148WS, Diode_SMD:D_SOD-323, symbol Diode:1N4148WS
- removed R40, R41, R46, R47: 100R, Resistor_SMD:R_0603_1608Metric, symbol Device:R
- removed R43, R48, R49: 1k, Resistor_SMD:R_0603_1608Metric, symbol Device:R
- added R26, R28, R30, R32: 2k, Resistor_SMD:R_0603_1608Metric, symbol Device:R
- added R27, R29, R31: 1k, Resistor_SMD:R_0603_1608Metric, symbol Device:R
Connections:
- net +5V: no longer R42.1
- net GND: now also R26.2, R28.2, R30.2, R32.2
- net TRM1_SUB: now also R42.1
- net TRM2_SUB: now also R27.1
- net TRM3_SUB: now also R29.1
- net TRM4_SUB: now also R31.1
- net V_SW_SUB: now also U6.11 (+), U6.5 (+), U6.7 (+), U6.9 (+); no longer U6.10 (-), U6.4 (-), U6.6 (-), U6.8 (-)
- net at R42.2: now also U6.4 (-), R26.1
- new net: R29.2, R30.1, U6.8 (-)
- new net: R31.2, R32.1, U6.10 (-)
- new net: R27.2, R28.1, U6.6 (-)
Other:
- title: IO_16x8_matrix -> Opto_8
