File: Opto_8/rtn_sub_4x.kicad_sch (KiCad schematic)
At the start: 15 parts, among them U7 LM339

Commit message: configurable_inputs
Parts:
- renumbered R39 to R47, R40 to R48, R41 to R49, R42 to R50, R43 to R51, R44 to R52, R45 to R53, R46 to R54, R47 to R55, R48 to R56, R49 to R57, R50 to R58
Changed lines of the file:
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@@
   (symbol (lib_id "Device:R") (at 71.12 96.52 0) (unit 1)
     (in_bom yes) (on_board yes)
-    (property "Reference" "R40" (id 0) (at 71.12 97.79 90)
+    (property "Reference" "R48" (id 0) (at 71.12 97.79 90)
       (effects (font (size 1.27 1.27)) (justify left))
     )
@@
   (symbol (lib_id "power:GND") (at 104.14 62.23 0) (unit 1)
     (in_bom yes) (on_board yes)
-    (property "Reference" "#PWR074" (id 0) (at 104.14 68.58 0)
+    (property "Reference" "#PWR084" (id 0) (at 104.14 68.58 0)
       (effects (font (size 1.27 1.27)) hide)
     )
@@
   (symbol (lib_id "power:GND") (at 81.28 172.72 0) (unit 1)
     (in_bom yes) (on_board yes)
-    (property "Reference" "#PWR073" (id 0) (at 81.28 179.07 0)
+    (property "Reference" "#PWR083" (id 0) (at 81.28 179.07 0)
       (effects (font (size 1.27 1.27)) hide)
     )
@@
   (symbol (lib_id "power:+3V3") (at 71.12 91.44 0) (unit 1)
     (in_bom yes) (on_board yes)
-    (property "Reference" "#PWR071" (id 0) (at 71.12 95.25 0)
+    (property "Reference" "#PWR081" (id 0) (at 71.12 95.25 0)
       (effects (font (size 1.27 1.27)) hide)
     )
@@
   (symbol (lib_id "power:GND") (at 208.28 62.23 0) (unit 1)
     (in_bom yes) (on_board yes)
-    (property "Reference" "#PWR079" (id 0) (at 208.28 68.58 0)
+    (property "Reference" "#PWR089" (id 0) (at 208.28 68.58 0)
       (effects (font (size 1.27 1.27)) hide)
     )
@@
   (symbol (lib_id "Device:R") (at 104.14 46.99 0) (unit 1)
     (in_bom yes) (on_board yes) (fields_autoplaced)
-    (property "Reference" "R41" (id 0) (at 106.68 45.7199 0)
+    (property "Reference" "R49" (id 0) (at 106.68 45.7199 0)
       (effects (font (size 1.27 1.27)) (justify left))
     )
@@
   (symbol (lib_id "power:+3V3") (at 71.12 41.91 0) (unit 1)
     (in_bom yes) (on_board yes)
-    (property "Reference" "#PWR070" (id 0) (at 71.12 45.72 0)
+    (property "Reference" "#PWR080" (id 0) (at 71.12 45.72 0)
       (effects (font (size 1.27 1.27)) hide)
     )
@@
   (symbol (lib_id "Device:R") (at 175.26 46.99 0) (unit 1)
     (in_bom yes) (on_board yes)
-    (property "Reference" "R45" (id 0) (at 175.26 48.26 90)
+    (property "Reference" "R53" (id 0) (at 175.26 48.26 90)
       (effects (font (size 1.27 1.27)) (justify left))
     )
@@
   (symbol (lib_id "Device:R") (at 208.28 106.68 0) (unit 1)
     (in_bom yes) (on_board yes) (fields_autoplaced)
-    (property "Reference" "R50" (id 0) (at 210.82 105.4099 0)
+    (property "Reference" "R58" (id 0) (at 210.82 105.4099 0)
       (effects (font (size 1.27 1.27)) (justify left))
     )
@@
   (symbol (lib_id "power:GND") (at 110.49 172.72 0) (unit 1)
     (in_bom yes) (on_board yes)
-    (property "Reference" "#PWR076" (id 0) (at 110.49 179.07 0)
+    (property "Reference" "#PWR086" (id 0) (at 110.49 179.07 0)
       (effects (font (size 1.27 1.27)) hide)
     )
@@
   (symbol (lib_id "power:+3V3") (at 175.26 91.44 0) (unit 1)
     (in_bom yes) (on_board yes)
-    (property "Reference" "#PWR078" (id 0) (at 175.26 95.25 0)
+    (property "Reference" "#PWR088" (id 0) (at 175.26 95.25 0)
       (effects (font (size 1.27 1.27)) hide)
     )
@@
   (symbol (lib_id "Device:R") (at 208.28 96.52 0) (unit 1)
     (in_bom yes) (on_board yes) (fields_autoplaced)
-    (property "Reference" "R49" (id 0) (at 210.82 95.2499 0)
+    (property "Reference" "R57" (id 0) (at 210.82 95.2499 0)
       (effects (font (size 1.27 1.27)) (justify left))
     )
@@
   (symbol (lib_id "Device:R") (at 208.28 57.15 0) (unit 1)
     (in_bom yes) (on_board yes) (fields_autoplaced)
-    (property "Reference" "R48" (id 0) (at 210.82 55.8799 0)
+    (property "Reference" "R56" (id 0) (at 210.82 55.8799 0)
       (effects (font (size 1.27 1.27)) (justify left))
     )
@@
   (symbol (lib_id "power:GND") (at 104.14 111.76 0) (unit 1)
     (in_bom yes) (on_board yes)
-    (property "Reference" "#PWR075" (id 0) (at 104.14 118.11 0)
+    (property "Reference" "#PWR085" (id 0) (at 104.14 118.11 0)
       (effects (font (size 1.27 1.27)) hide)
     )
@@
   (symbol (lib_id "Device:R") (at 71.12 46.99 0) (unit 1)
     (in_bom yes) (on_board yes)
-    (property "Reference" "R39" (id 0) (at 71.12 48.26 90)
+    (property "Reference" "R47" (id 0) (at 71.12 48.26 90)
       (effects (font (size 1.27 1.27)) (justify left))
     )
@@
   (symbol (lib_id "Device:R") (at 104.14 106.68 0) (unit 1)
     (in_bom yes) (on_board yes) (fields_autoplaced)
-    (property "Reference" "R44" (id 0) (at 106.68 105.4099 0)
+    (property "Reference" "R52" (id 0) (at 106.68 105.4099 0)
       (effects (font (size 1.27 1.27)) (justify left))
     )
@@
   (symbol (lib_id "power:+3V3") (at 175.26 41.91 0) (unit 1)
     (in_bom yes) (on_board yes)
-    (property "Reference" "#PWR077" (id 0) (at 175.26 45.72 0)
+    (property "Reference" "#PWR087" (id 0) (at 175.26 45.72 0)
       (effects (font (size 1.27 1.27)) hide)
     )
@@
   (symbol (lib_id "Device:R") (at 104.14 57.15 0) (unit 1)
     (in_bom yes) (on_board yes) (fields_autoplaced)
-    (property "Reference" "R42" (id 0) (at 106.68 55.8799 0)
+    (property "Reference" "R50" (id 0) (at 106.68 55.8799 0)
       (effects (font (size 1.27 1.27)) (justify left))
     )
@@
   (symbol (lib_id "Device:R") (at 104.14 96.52 0) (unit 1)
     (in_bom yes) (on_board yes) (fields_autoplaced)
-    (property "Reference" "R43" (id 0) (at 106.68 95.2499 0)
+    (property "Reference" "R51" (id 0) (at 106.68 95.2499 0)
       (effects (font (size 1.27 1.27)) (justify left))
     )
@@
   (symbol (lib_id "Device:R") (at 208.28 46.99 0) (unit 1)
     (in_bom yes) (on_board yes) (fields_autoplaced)
-    (property "Reference" "R47" (id 0) (at 210.82 45.7199 0)
+    (property "Reference" "R55" (id 0) (at 210.82 45.7199 0)
       (effects (font (size 1.27 1.27)) (justify left))
     )
@@
   (symbol (lib_id "Device:R") (at 175.26 96.52 0) (unit 1)
     (in_bom yes) (on_board yes)
-    (property "Reference" "R46" (id 0) (at 175.26 97.79 90)
+    (property "Reference" "R54" (id 0) (at 175.26 97.79 90)
       (effects (font (size 1.27 1.27)) (justify left))
     )
@@
   (symbol (lib_id "power:+5V") (at 81.28 152.4 0) (unit 1)
     (in_bom yes) (on_board yes)
-    (property "Reference" "#PWR072" (id 0) (at 81.28 156.21 0)
+    (property "Reference" "#PWR082" (id 0) (at 81.28 156.21 0)
       (effects (font (size 1.27 1.27)) hide)
     )
@@
   (symbol (lib_id "power:GND") (at 208.28 111.76 0) (unit 1)
     (in_bom yes) (on_board yes)
-    (property "Reference" "#PWR080" (id 0) (at 208.28 118.11 0)
-      (effects (font (size 1.27 1.27)) hide)
-    )
+    (property "Reference" "#PWR090" (id 0) (at 208.28 118.11 0)
+      (effects (font (size 1.27 1.27)) hide)
+    )
