File: Opto_8/Drv8.kicad_sch (KiCad schematic)
At the start: 34 parts, among them J5 Conn_01x09, J6 Conn_01x09, Q1 MMBT3904, Q2 MMBT3904, Q3 MMBT3904, Q4 MMBT3904, Q5 MMBT3904, Q6 MMBT3904, Q7 MMBT3904, Q8 MMBT3904

Commit message: in16_drv8
Parts:
- removed C25, C26, C27, C28, C29, C30, C31, C32: 10n, Capacitor_SMD:C_0603_1608Metric, symbol Device:C
- removed J5: Conn_01x09, Connector_Molex:Molex_KK-254_AE-6410-09A_1x09_P2.54mm_Vertical, symbol Connector_Generic:Conn_01x09
- removed J6: Conn_01x09, Connector_Molex:Molex_KK-396_5273-09A_1x09_P3.96mm_Vertical, symbol Connector_Generic:Conn_01x09
- removed Q1, Q2, Q3, Q4, Q5, Q6, Q7, Q8: MMBT3904, Package_TO_SOT_SMD:SOT-23, symbol Transistor_BJT:MMBT3904
- removed R26, R27, R28, R29, R30, R31, R32, R33, R34, R35: 1k, Resistor_SMD:R_0603_1608Metric, symbol Device:R
- added J5: Conn_01x10, symbol Connector_Generic:Conn_01x10
- added R3, R5: 180R, Resistor_SMD:R_1206_3216Metric, symbol Device:R
- R20, R21, R22, R23, R24, R25: value 1k -> 180R; footprint Resistor_SMD:R_0603_1608Metric -> Resistor_SMD:R_1206_3216Metric
Connections:
- net DRV_1 is gone; now on net +5V: R20.1
- net DRV_2 is gone; now on net +5V: R21.1
- net DRV_3 is gone; now on net +5V: R22.1
- net DRV_4 is gone; now on net +5V: R23.1
- net +5V: now also R3.1, R5.1
- net D1: now also J5.1 (Pin_1)
- net D2: now also J5.2 (Pin_2), R3.2; no longer R25.2
- net D3: now also J5.3 (Pin_3), R5.2
- net D4: now also R20.2, J5.4 (Pin_4)
- net D5: now also R21.2, J5.5 (Pin_5)
- net D6: now also R22.2, J5.6 (Pin_6)
- net D7: now also R23.2, J5.7 (Pin_7)
- net D8: now also R25.2, J5.9 (Pin_9)
- net GND: now also J5.10 (Pin_10)
- no-connect marks 2 -> 1
Other:
- note removed: "Stern S.A.M. connector"
- note removed: "WPC connector"
- title: IO_16x8_matrix -> Opto_8

Commit message: basic
Parts:
- added J10, J11, J12, J13, J6, J7, J8, J9: Conn_01x02, Connector_Molex:Molex_KK-254_AE-6410-02A_1x02_P2.54mm_Vertical, symbol Connector_Generic:Conn_01x02
- J5: footprint (none) -> Connector_Molex:Molex_KK-254_AE-6410-10A_1x10_P2.54mm_Vertical
- renumbered R24 to R27, R3 to R28, R5 to R29, R20 to R30, R21 to R31, R22 to R32, R23 to R33, R25 to R34
Connections:
- net D1: now also J6.1 (Pin_1)
- net D2: now also J7.1 (Pin_1)
- net D3: now also J8.1 (Pin_1)
- net D4: now also J9.1 (Pin_1)
- net D5: now also J10.1 (Pin_1)
- net D6: now also J11.1 (Pin_1)
- net D7: now also J12.1 (Pin_1)
- net D8: now also J13.1 (Pin_1)
- net GND: now also J10.2 (Pin_2), J11.2 (Pin_2), J12.2 (Pin_2), J13.2 (Pin_2), J6.2 (Pin_2), J7.2 (Pin_2), J8.2 (Pin_2), J9.2 (Pin_2)
