File: Opto_8/In16.kicad_sch (KiCad schematic)
At the start: 6 parts, among them J7 Conn_01x09, J8 Conn_01x10, J9 Conn_01x10

Commit message: in16_drv8
Parts:
- R37: value 2k -> 1k
Other:
- title: IO_16x8_matrix -> Opto_8
Changed lines of the file:
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@@
   (paper "A4")
   (title_block
-    (title "IO_16x8_matrix")
-    (date "2024-12-01")
-    (rev "1.0.0")
+    (title "Opto_8")
+    (date "2025-03-26")
+    (rev "0.1.0")
   )
   (junction (at 209.55 118.11) (diameter 0) (color 0 0 0 0)
@@
       (effects (font (size 1.27 1.27)) (justify left))
     )
-    (property "Value" "2k" (id 1) (at 212.09 124.4599 0)
+    (property "Value" "1k" (id 1) (at 212.09 124.4599 0)
       (effects (font (size 1.27 1.27)) (justify left))
     )

Commit message: basic
Parts:
- removed J7: Conn_01x09, Connector_Molex:Molex_KK-254_AE-6410-09A_1x09_P2.54mm_Vertical, symbol Connector_Generic:Conn_01x09
- removed J8, J9: Conn_01x10, Connector_Molex:Molex_KK-396_5273-10A_1x10_P3.96mm_Vertical, symbol Connector_Generic:Conn_01x10
- added C27: 10u, Capacitor_SMD:C_0603_1608Metric, symbol Device:C
- added J14: Conn_01x10, Connector_Molex:Molex_KK-254_AE-6410-10A_1x10_P2.54mm_Vertical, symbol Connector_Generic:Conn_01x10
- added R37: 330k, Resistor_SMD:R_0603_1608Metric, symbol Device:R
- added R38: 6k8, Resistor_SMD:R_0603_1608Metric, symbol Device:R
- renumbered C33 to C26, R36 to R35, R37 to R36
Connections:
- net +5V: now also J14.1 (Pin_1), R37.1
- net GND: now also C27.2, R38.2
- net T1: now also J14.10 (Pin_10)
- net T2: now also J14.9 (Pin_9)
- net T3: now also J14.8 (Pin_8)
- net T4: now also J14.7 (Pin_7)
- net T5: now also J14.6 (Pin_6)
- net T6: now also J14.4 (Pin_4)
- net T7: now also J14.3 (Pin_3)
- net T8: now also J14.2 (Pin_2)
- new net V_SW_D: C27.1, R37.2, R38.1
- no-connect marks 5 -> 1
Other:
- sheet 3_RTN_SUB_4x renamed 1_RDI_SUB_4x
- sheet 4_RTN_SUB_4x renamed 2_RDI_SUB_4x
- sheet 1_RDI_SUB_4x: file rtn_sub_4x.kicad_sch -> rdi_sub_4x.kicad_sch
- sheet 2_RDI_SUB_4x: file rtn_sub_4x.kicad_sch -> rdi_sub_4x.kicad_sch
- note added: "Photo Diodes"
- note added: "Photo Transistors"
- note removed: "Stern S.A.M. connector"
- note removed: "WPC connector"
- moved on the sheet: C26, R35, R36

Commit message: configurable_inputs
Parts:
- added J15: Conn_01x10, Connector_Molex:Molex_KK-254_AE-6410-10A_1x10_P2.54mm_Vertical, symbol Connector_Generic:Conn_01x10
- added JP2: open: LED, closed: Transistor, Connector_PinHeader_2.54mm:PinHeader_1x02_P2.54mm_Vertical, symbol Jumper:Jumper_2_Open
- renumbered J14 to J16, R35 to R43, R36 to R44, R37 to R45, R38 to R46
Connections:
- net +5V: now also J15.1 (Pin_1)
- net T1: now also J15.10 (Pin_10); no longer J16.10 (Pin_10)
- net T10: now also J16.3 (Pin_3)
- net T11: now also J16.5 (Pin_5)
- net T12: now also J16.6 (Pin_6)
- net T13: now also J16.7 (Pin_7)
- net T14: now also J16.8 (Pin_8)
- net T15: now also J16.9 (Pin_9)
- net T16: now also J16.10 (Pin_10)
- net T2: now also J15.9 (Pin_9); no longer J16.9 (Pin_9)
- net T3: now also J15.8 (Pin_8); no longer J16.8 (Pin_8)
- net T4: now also J15.7 (Pin_7); no longer J16.7 (Pin_7)
- net T5: now also J15.6 (Pin_6); no longer J16.6 (Pin_6)
- net T6: now also J15.4 (Pin_4); no longer J16.4 (Pin_4)
- net T7: now also J15.3 (Pin_3); no longer J16.3 (Pin_3)
- net T8: now also J15.2 (Pin_2); no longer J16.2 (Pin_2)
- net T9: now also J16.2 (Pin_2)
- net V_SWITCH: now also JP2.1 (A)
- net V_SW_D: now also JP2.2 (B)
- no-connect marks 1 -> 2
