File: Opto_8/Opto_8.kicad_pcb (KiCad board)
At the start: 2 copper layers, 97.6 x 67.3 mm, 210 parts, among them J1 Conn_01x06, J2 nmount SW Debug, J3 USB_C_Receptacle_USB2.0, J4 Conn_01x06, J5 Conn_01x09, J6 Conn_01x09, J7 Conn_01x09, J8 Conn_01x10, J9 Conn_01x10, Q1 MMBT3904, Q2 MMBT3904, Q3 MMBT3904, Q4 MMBT3904, Q5 MMBT3904, Q6 MMBT3904, Q7 MMBT3904, Q8 MMBT3904, SW1 Reset, SW2 Boot, SW3 ADDRESS, U1 ADM3483, U14 LMV321, U2 W25Q128JVSIQ, U3 RP2040, U4 SN74AHCT1G125, U5 AP2112K-3.3, U6 LM339, U7 LM339, U8 LM339, U9 LM339, Y1 12MHz,18pF

Commit message: basic
Parts:
- removed the C25 at (182.5, 60.5)
- removed the C26 at (182.5, 64.1)
- removed the C28 at (182.5, 71.6)
- removed the C29 at (182.5, 75.2)
- removed the C30 at (182.6, 79.0)
- removed the C31 at (192.8, 96.5)
- removed C36, C38, C39, C41, C43, C45, C46, C47, C48, C49, C50, C51, C52, C53, C54, C55, C56, C57, C58: 100n, Capacitor_SMD:C_0402_1005Metric
- removed D10, D11, D12, D13, D14, D15, D16, D17, D18, D19, D20, D21, D22, D8, D9: 1N4148WS, Diode_SMD:D_SOD-323
- removed the D7 at (106.7, 60.3)
- removed Q1, Q2, Q3, Q4, Q5, Q6, Q7, Q8: MMBT3904, Package_TO_SOT_SMD:SOT-23
- removed the R20 at (176.1, 61.3)
- removed the R21 at (176.1, 65.2)
- removed the R22 at (176.1, 68.8)
- removed the R23 at (176.1, 72.5)
- removed the R25 at (182.5, 65.8)
- removed the R26 at (182.5, 69.5)
- removed the R27 at (182.5, 73.3)
- removed the R35 at (192.8, 94.6)
- removed the R40 at (112.9, 60.2)
- removed the R41 at (112.9, 62.4)
- removed the R46 at (112.9, 64.6)
- removed the R52 at (112.9, 70.2)
- removed the R53 at (112.9, 72.1)
- removed R79, R80, R85, R86, R91, R92: 100R, Resistor_SMD:R_0603_1608Metric
- removed R81, R82, R87, R88, R93, R94: 1k, Resistor_SMD:R_0603_1608Metric
- removed R83, R84, R89, R90: 10k, Resistor_SMD:R_0603_1608Metric
- removed REF** (x3): MountingHole_5.5mm_Pinball, IO_16x8_matrix:MountingHole_5.5mm_Pinball
- removed the U8 at (120.3, 83.8)
- added C33: 100n, Capacitor_SMD:C_0402_1005Metric, F.Cu at (113.1, 158.7)
- added C34: 100n, Capacitor_SMD:C_0402_1005Metric, F.Cu at (143.8, 128.5)
- added J10: Conn_01x02, Connector_Molex:Molex_KK-254_AE-6410-02A_1x02_P2.54mm_Vertical, F.Cu at (225.3, 65.9)
- added J11: Conn_01x02, Connector_Molex:Molex_KK-254_AE-6410-02A_1x02_P2.54mm_Vertical, F.Cu at (217.4, 65.9)
- added J12: Conn_01x02, Connector_Molex:Molex_KK-254_AE-6410-02A_1x02_P2.54mm_Vertical, F.Cu at (225.3, 58.7)
- added J13: Conn_01x02, Connector_Molex:Molex_KK-254_AE-6410-02A_1x02_P2.54mm_Vertical, F.Cu at (225.3, 80.1)
- added J14: Conn_01x10, Connector_Molex:Molex_KK-254_AE-6410-10A_1x10_P2.54mm_Vertical, F.Cu at (132.3, 116.7)
- added J15: Conn_01x02, Connector_Molex:Molex_KK-254_AE-6410-02A_1x02_P2.54mm_Vertical, F.Cu at (168.3, 125.8)
- added J16: Conn_01x02, Connector_Molex:Molex_KK-254_AE-6410-02A_1x02_P2.54mm_Vertical, F.Cu at (175.4, 125.8)
- added J17: Conn_01x02, Connector_Molex:Molex_KK-254_AE-6410-02A_1x02_P2.54mm_Vertical, F.Cu at (182.5, 125.8)
- added J18: Conn_01x02, Connector_Molex:Molex_KK-254_AE-6410-02A_1x02_P2.54mm_Vertical, F.Cu at (182.5, 118.0)
- added J19: Conn_01x02, Connector_Molex:Molex_KK-254_AE-6410-02A_1x02_P2.54mm_Vertical, F.Cu at (168.3, 145.0)
- added J20: Conn_01x02, Connector_Molex:Molex_KK-254_AE-6410-02A_1x02_P2.54mm_Vertical, F.Cu at (175.4, 145.0)
- added J21: Conn_01x02, Connector_Molex:Molex_KK-254_AE-6410-02A_1x02_P2.54mm_Vertical, F.Cu at (182.5, 145.0)
- added J22: Conn_01x02, Connector_Molex:Molex_KK-254_AE-6410-02A_1x02_P2.54mm_Vertical, F.Cu at (182.5, 137.1)
- added R37: 330k, Resistor_SMD:R_0603_1608Metric, F.Cu at (93.2, 134.1)
- added R38: 6k8, Resistor_SMD:R_0603_1608Metric, F.Cu at (97.2, 134.1)
- added R42: 2k, Resistor_SMD:R_0603_1608Metric, F.Cu at (131.9, 155.0)
- added R44: 2k, Resistor_SMD:R_0603_1608Metric, F.Cu at (127.9, 157.5)
- added R50: 2k, Resistor_SMD:R_0603_1608Metric, F.Cu at (127.9, 152.5)
- added R54: 2k, Resistor_SMD:R_0603_1608Metric, F.Cu at (131.9, 142.8)
- added R56: 2k, Resistor_SMD:R_0603_1608Metric, F.Cu at (127.9, 145.3)
- added R59: 1k, Resistor_SMD:R_0603_1608Metric, F.Cu at (131.9, 145.3)
- added R60: 2k, Resistor_SMD:R_0603_1608Metric, F.Cu at (131.9, 140.3)
- added R61: 1k, Resistor_SMD:R_0603_1608Metric, F.Cu at (127.9, 142.8)
- added R62: 2k, Resistor_SMD:R_0603_1608Metric, F.Cu at (127.9, 140.3)
- added R63: 10k, Resistor_SMD:R_0603_1608Metric, F.Cu at (105.7, 164.0)
- added R64: 10k, Resistor_SMD:R_0603_1608Metric, F.Cu at (109.7, 159.0)
- added R65: 1M, Resistor_SMD:R_0603_1608Metric, F.Cu at (105.7, 159.0)
- added R66: 1M, Resistor_SMD:R_0603_1608Metric, F.Cu at (101.7, 166.5)
- added U10: LM339, Package_SO:SOIC-14_3.9x8.7mm_P1.27mm, F.Cu at (130.2, 130.1)
- C27: value 10n -> 10u
- C32: value 10n -> 100n; footprint Capacitor_SMD:C_0603_1608Metric -> Capacitor_SMD:C_0402_1005Metric
- J5: value Conn_01x09 -> Conn_01x10; footprint Connector_Molex:Molex_KK-254_AE-6410-09A_1x09_P2.54mm_Vertical -> Connector_Molex:Molex_KK-254_AE-6410-10A_1x10_P2.54mm_Vertical
- J6: value Conn_01x09 -> Conn_01x02; footprint Connector_Molex:Molex_KK-396_5273-09A_1x09_P3.96mm_Vertical -> Connector_Molex:Molex_KK-254_AE-6410-02A_1x02_P2.54mm_Vertical
- J7: value Conn_01x09 -> Conn_01x02; footprint Connector_Molex:Molex_KK-254_AE-6410-09A_1x09_P2.54mm_Vertical -> Connector_Molex:Molex_KK-254_AE-6410-02A_1x02_P2.54mm_Vertical
- J8, J9: value Conn_01x10 -> Conn_01x02; footprint Connector_Molex:Molex_KK-396_5273-10A_1x10_P3.96mm_Vertical -> Connector_Molex:Molex_KK-254_AE-6410-02A_1x02_P2.54mm_Vertical
- R27: renamed from R24; value 1k -> 180R; footprint Resistor_SMD:R_0603_1608Metric -> Resistor_SMD:R_1206_3216Metric
- R28, R29, R30, R31, R32, R33, R34: value 1k -> 180R; footprint Resistor_SMD:R_0603_1608Metric -> Resistor_SMD:R_1206_3216Metric
- R36: renamed from R37; value 2k -> 1k
- R47: value 100R -> 1k
- R48: value 1k -> 2k
- R67, R68: value 100R -> 10k
- R69, R70: value 1k -> 1M
- R73, R74: value 100R -> 1M
- R75, R76: value 1k -> 10k
- R77, R78: value 10k -> 1M
- moved R32 116.1 mm to (94.0, 151.9), turned to 0 degrees
- moved R28 109.5 mm to (94.0, 148.6), turned to 0 degrees
- moved J7 109.1 mm to (217.4, 80.1), turned to -90 degrees
- moved C32 108.1 mm to (109.1, 161.2)
- moved R33 107.2 mm to (99.6, 148.6), turned to 0 degrees
- moved R30 102.4 mm to (99.6, 151.9), turned to 0 degrees
- moved R31 99.8 mm to (105.2, 151.9), turned to 0 degrees
- moved R29 98.9 mm to (105.2, 148.6), turned to 0 degrees
- moved R34 96.2 mm to (110.8, 148.6), turned to 0 degrees
- moved R43 94.1 mm to (136.0, 152.5)
- moved R47 92.9 mm to (131.9, 157.5), turned to 0 degrees
- moved J8 91.2 mm to (217.4, 58.7), turned to -90 degrees
- moved R48 90.6 mm to (131.9, 152.5)
- moved R49 90.1 mm to (127.9, 155.0)
- moved R70 88.1 mm to (101.7, 164.0)
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- renumbered C9 to C10, C10 to C11, C11 to C12, C12 to C13, C13 to C14, C14 to C15, C15 to C16, C16 to C17, C17 to C18, C18 to C19, C19 to C20, C20 to C21, C21 to C22, C22 to C23, C23 to C24, C24 to C25, C33 to C26, C34 to C28, C37 to C29, C40 to C30, C44 to C31, C42 to C8, C8 to C9, D23 to D7, R12 to R10, R13 to R11, R14 to R12, R56 to R13, R57 to R14, R58 to R15, R15 to R16, R59 to R17, R60 to R18, R61 to R19, R62 to R20, R63 to R21, R64 to R22, R16 to R23, R17 to R24, R18 to R25, R19 to R26, R4 to R3, R36 to R35, R38 to R39, R6 to R4, R39 to R40, R42 to R41, R44 to R45, R45 to R46, R7 to R5, R50 to R51, R51 to R52, R54 to R53, R65 to R57, R66 to R58, R8 to R6, R9 to R7, R10 to R8, R11 to R9, TP4 to TP1, TP5 to TP2, U14 to U3, U3 to U4, U4 to U5, U5 to U6, U6 to U7, U7 to U8
Connections:
- C27 pad 1: /Driver8/D3 -> /In16/V_SW_D
- C32 pad 1: /Driver8/D8 -> +5V
- C35 pad 1: Net-(C35-Pad1) -> /In16/V_SW_D
- J6 pad 2: unconnected-(J6-Pad2) -> GND
- J7 pad 1: /In16/T1 -> /Driver8/D2
- J7 pad 2: /In16/T2 -> GND
- J8 pad 1: /In16/T8 -> /Driver8/D3
- J8 pad 2: /In16/T7 -> GND
- J9 pad 1: /In16/T16 -> /Driver8/D4
- J9 pad 2: /In16/T15 -> GND
- R28 pad 1: /Out_5 -> +5V
- R28 pad 2: Net-(Q5-Pad1) -> /Driver8/D2
- R29 pad 1: /Out_6 -> +5V
- R29 pad 2: Net-(Q6-Pad1) -> /Driver8/D3
- R30 pad 1: /Out_7 -> +5V
- R30 pad 2: Net-(Q7-Pad1) -> /Driver8/D4
- R31 pad 1: /Out_8 -> +5V
- R31 pad 2: Net-(Q8-Pad1) -> /Driver8/D5
- R32 pad 2: /Driver8/D5 -> /Driver8/D6
- R33 pad 2: /Driver8/D6 -> /Driver8/D7
- R34 pad 2: /Driver8/D7 -> /Driver8/D8
- R41 pad 1: +5V -> /In16/T1
- R41 pad 2: Net-(D7-Pad2) -> Net-(R42-Pad1)
- R43 pad 1: +5V -> /In16/T2
- R43 pad 2: Net-(D8-Pad2) -> Net-(R43-Pad2)
- R47 pad 1: Net-(C39-Pad1) -> /In16/T3
- R47 pad 2: Net-(D10-Pad2) -> Net-(R47-Pad2)
- R48 pad 1: +5V -> Net-(R47-Pad2)
- R48 pad 2: Net-(D9-Pad2) -> GND
- R49 pad 1: +5V -> /In16/T4
- R49 pad 2: Net-(D10-Pad2) -> Net-(R49-Pad2)
- R53 pad 1: +5V -> /In16/T5
- R53 pad 2: Net-(D11-Pad2) -> Net-(R53-Pad2)
- R55 pad 1: +5V -> /In16/T6
- R55 pad 2: Net-(D12-Pad2) -> Net-(R55-Pad2)
- R67 pad 1: Net-(C45-Pad1) -> +3V3
- R67 pad 2: Net-(D13-Pad2) -> /In_11
- R68 pad 1: Net-(C46-Pad1) -> +3V3
- R68 pad 2: Net-(D14-Pad2) -> /In_12
- R69 pad 1: +5V -> /In16/T11
- R69 pad 2: Net-(D13-Pad2) -> GND
- R70 pad 1: +5V -> /In16/T12
- R70 pad 2: Net-(D14-Pad2) -> GND
- R71 pad 2: /In_9 -> /In_13
- R72 pad 2: /In_10 -> /In_14
- R73 pad 1: Net-(C48-Pad1) -> /In16/T13
- R73 pad 2: Net-(D15-Pad2) -> GND
- R74 pad 1: Net-(C49-Pad1) -> /In16/T14
- R74 pad 2: Net-(D16-Pad2) -> GND
- R75 pad 1: +5V -> +3V3
- R75 pad 2: Net-(D15-Pad2) -> /In_15
- R76 pad 1: +5V -> +3V3
- R76 pad 2: Net-(D16-Pad2) -> /In_16
- R77 pad 1: +3V3 -> /In16/T15
- R77 pad 2: /In_11 -> GND
- R78 pad 1: +3V3 -> /In16/T16
- R78 pad 2: /In_12 -> GND
- U4 pad 30: /Out_8 -> unconnected-(U4-Pad30)
- U4 pad 31: /Out_7 -> unconnected-(U4-Pad31)
- U4 pad 32: /Out_6 -> unconnected-(U4-Pad32)
- U4 pad 34: /Out_5 -> unconnected-(U4-Pad34)
- U4 pad 35: /Out_4 -> unconnected-(U4-Pad35)
- U4 pad 36: /Out_3 -> unconnected-(U4-Pad36)
- U4 pad 38: /Out_2 -> unconnected-(U4-Pad38)
- U4 pad 39: /Out_1 -> unconnected-(U4-Pad39)
- U7 pad 10: /In16/V_SWITCH -> Net-(R49-Pad2)
- U7 pad 11: Net-(C39-Pad1) -> /In16/V_SWITCH
- U7 pad 4: /In16/V_SWITCH -> Net-(R42-Pad1)
- U7 pad 5: Net-(C35-Pad1) -> /In16/V_SWITCH
- U7 pad 6: /In16/V_SWITCH -> Net-(R43-Pad2)
- U7 pad 7: Net-(C36-Pad1) -> /In16/V_SWITCH
- U7 pad 8: /In16/V_SWITCH -> Net-(R47-Pad2)
- U7 pad 9: Net-(C38-Pad1) -> /In16/V_SWITCH
- U8 pad 10: /In16/V_SWITCH -> Net-(R61-Pad2)
- U8 pad 11: Net-(C46-Pad1) -> /In16/V_SWITCH
- U8 pad 4: /In16/V_SWITCH -> Net-(R53-Pad2)
- U8 pad 5: Net-(C41-Pad1) -> /In16/V_SWITCH
- U8 pad 6: /In16/V_SWITCH -> Net-(R55-Pad2)
- U8 pad 7: Net-(C43-Pad1) -> /In16/V_SWITCH
- U8 pad 8: /In16/V_SWITCH -> Net-(R59-Pad2)
- U8 pad 9: Net-(C45-Pad1) -> /In16/V_SWITCH
- U9 pad 1: /In_14 -> /In_10
- U9 pad 10: /In16/V_SWITCH -> /In16/T12
- U9 pad 11: Net-(C58-Pad1) -> /In16/V_SW_D
- U9 pad 13: /In_16 -> /In_12
- U9 pad 14: /In_15 -> /In_11
- U9 pad 2: /In_13 -> /In_9
- U9 pad 4: /In16/V_SWITCH -> /In16/T9
- U9 pad 5: Net-(C54-Pad1) -> /In16/V_SW_D
- U9 pad 6: /In16/V_SWITCH -> /In16/T10
- U9 pad 7: Net-(C55-Pad1) -> /In16/V_SW_D
- U9 pad 8: /In16/V_SWITCH -> /In16/T11
- U9 pad 9: Net-(C57-Pad1) -> /In16/V_SW_D
Routing:
- net (no net): track 0.00 -> 139.4 mm
- net unconnected-(U4-Pad31): track 0.00 -> 56.7 mm, vias 0 -> 2
- net /Out_7: track 56.7 -> 0.00 mm, vias 2 -> 0
- net unconnected-(U4-Pad30): track 0.00 -> 53.5 mm, vias 0 -> 2
- net /Out_8: track 53.5 -> 0.00 mm, vias 2 -> 0
- net /In16/V_SWITCH: track 96.4 -> 144.4 mm
- net unconnected-(U4-Pad36): track 0.00 -> 44.8 mm, vias 0 -> 2
- net /Out_3: track 44.8 -> 0.00 mm, vias 2 -> 0
- net unconnected-(U4-Pad39): track 0.00 -> 44.2 mm, vias 0 -> 2
- net /Out_1: track 44.2 -> 0.00 mm, vias 2 -> 0
- net unconnected-(U4-Pad35): track 0.00 -> 42.7 mm, vias 0 -> 2
- net /Out_4: track 42.7 -> 0.00 mm, vias 2 -> 0
- net unconnected-(U4-Pad38): track 0.00 -> 41.4 mm, vias 0 -> 2
- net /Out_2: track 41.4 -> 0.00 mm, vias 2 -> 0
- net unconnected-(U4-Pad34): track 0.00 -> 39.7 mm, vias 0 -> 2
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
Commit message: configurable_inputs
Parts:
- added J15: Conn_01x10, Connector_Molex:Molex_KK-254_AE-6410-10A_1x10_P2.54mm_Vertical, F.Cu at (134.9, 117.8)
- added J5: Conn_01x10, Connector_Molex:Molex_KK-254_AE-6410-10A_1x10_P2.54mm_Vertical, F.Cu at (206.1, 84.6)
- added JP2: open: LED, closed: Transistor, Connector_PinHeader_2.54mm:PinHeader_1x02_P2.54mm_Vertical, F.Cu at (223.1, 126.0)
- added R35: 180R, Resistor_SMD:R_1206_3216Metric, F.Cu at (242.1, 80.0)
- added R36: 180R, Resistor_SMD:R_1206_3216Metric, F.Cu at (253.3, 83.3)
- added R37: 180R, Resistor_SMD:R_1206_3216Metric, F.Cu at (247.7, 80.0)
- added R38: 180R, Resistor_SMD:R_1206_3216Metric, F.Cu at (258.9, 83.3)
- added R39: 180R, Resistor_SMD:R_1206_3216Metric, F.Cu at (253.3, 80.0)
- added R40: 180R, Resistor_SMD:R_1206_3216Metric, F.Cu at (258.9, 80.0)
- added R41: 180R, Resistor_SMD:R_1206_3216Metric, F.Cu at (247.7, 83.3)
- added R42: 180R, Resistor_SMD:R_1206_3216Metric, F.Cu at (242.1, 83.3)
- added R73: 1k, Resistor_SMD:R_0603_1608Metric, F.Cu at (213.5, 138.5)
- added R75: 2k, Resistor_SMD:R_0603_1608Metric, F.Cu at (205.5, 141.0)
- added R76: 1M, Resistor_SMD:R_0603_1608Metric, F.Cu at (213.5, 136.0)
- added R77: 2k, Resistor_SMD:R_0603_1608Metric, F.Cu at (209.5, 141.0)
- added R80: 1M, Resistor_SMD:R_0603_1608Metric, F.Cu at (209.5, 136.0)
- added R81: 2k, Resistor_SMD:R_0603_1608Metric, F.Cu at (205.5, 138.5)
- added R82: 1M, Resistor_SMD:R_0603_1608Metric, F.Cu at (205.5, 136.0)
- added R83: 2k, Resistor_SMD:R_0603_1608Metric, F.Cu at (209.5, 138.5)
- added R86: 1k, Resistor_SMD:R_0603_1608Metric, F.Cu at (213.5, 127.4)
- added R88: 2k, Resistor_SMD:R_0603_1608Metric, F.Cu at (205.5, 129.9)
- added R89: 1M, Resistor_SMD:R_0603_1608Metric, F.Cu at (213.5, 124.9)
- added R90: 2k, Resistor_SMD:R_0603_1608Metric, F.Cu at (209.5, 129.9)
- added R93: 1M, Resistor_SMD:R_0603_1608Metric, F.Cu at (209.5, 124.9)
- added R94: 2k, Resistor_SMD:R_0603_1608Metric, F.Cu at (205.5, 127.4)
- added R95: 1M, Resistor_SMD:R_0603_1608Metric, F.Cu at (205.5, 124.9)
- added R96: 2k, Resistor_SMD:R_0603_1608Metric, F.Cu at (209.5, 127.4)
- moved R28 170.7 mm to (241.4, 62.4)
- moved R29 170.7 mm to (252.6, 62.4)
- moved R30 170.7 mm to (247.0, 65.6)
- moved R31 170.7 mm to (252.6, 65.6)
- moved R32 170.7 mm to (241.4, 65.6)
- moved R33 170.7 mm to (247.0, 62.4)
- moved R34 170.7 mm to (258.2, 62.4)
- moved J16 40.4 mm to (172.7, 116.8)
- moved J14 15.2 mm to (206.1, 57.0)
- renumbered J5 to J14, J14 to J16, J15 to J17, J16 to J18, J17 to J19, J18 to J20, J19 to J21, J20 to J22, J21 to J23, J22 to J24, R35 to R43, R36 to R44, R37 to R45, R38 to R46, R39 to R47, R40 to R48, R41 to R49, R42 to R50, R43 to R51, R44 to R52, R45 to R53, R46 to R54, R47 to R55, R48 to R56, R49 to R57, R50 to R58, R51 to R59, R52 to R60, R53 to R61, R54 to R62, R55 to R63, R56 to R64, R57 to R65, R58 to R66, R59 to R67, R60 to R68, R61 to R69, R62 to R70, R63 to R71, R64 to R72, R65 to R74, R67 to R78, R68 to R79, R71 to R84, R72 to R85, R73 to R87, R75 to R91, R76 to R92
Connections:
- J14 pad 1: /Driver8/D1 -> GND
- J14 pad 10: GND -> /Driver8/D16
- J14 pad 2: /Driver8/D2 -> unconnected-(J14-Pad2)
- J14 pad 3: /Driver8/D3 -> /Driver8/D9
- J14 pad 4: /Driver8/D4 -> /Driver8/D10
- J14 pad 5: /Driver8/D5 -> /Driver8/D11
- J14 pad 6: /Driver8/D6 -> /Driver8/D12
- J14 pad 7: /Driver8/D7 -> /Driver8/D13
- J14 pad 8: unconnected-(J5-Pad8) -> /Driver8/D14
- J14 pad 9: /Driver8/D8 -> /Driver8/D15
- J16 pad 10: /In16/T1 -> /In16/T16
- J16 pad 2: /In16/T8 -> /In16/T9
- J16 pad 3: /In16/T7 -> /In16/T10
- J16 pad 4: /In16/T6 -> unconnected-(J16-Pad4)
- J16 pad 5: unconnected-(J14-Pad5) -> /In16/T11
- J16 pad 6: /In16/T5 -> /In16/T12
- J16 pad 7: /In16/T4 -> /In16/T13
- J16 pad 8: /In16/T3 -> /In16/T14
- J16 pad 9: /In16/T2 -> /In16/T15
- J17 pad 1: /In16/T9 -> Net-(J17-Pad1)
- J17 pad 2: GND -> Net-(R74-Pad2)
- J18 pad 2: GND -> Net-(J18-Pad2)
- J19 pad 2: GND -> Net-(J19-Pad2)
- J20 pad 2: GND -> Net-(J20-Pad2)
- J21 pad 1: /In16/T13 -> Net-(J21-Pad1)
- J21 pad 2: GND -> Net-(R87-Pad2)
- J22 pad 2: GND -> Net-(J22-Pad2)
- J23 pad 2: GND -> Net-(J23-Pad2)
- J24 pad 2: GND -> Net-(J24-Pad2)
- R74 pad 1: /In16/T9 -> Net-(J17-Pad1)
- R74 pad 2: GND -> Net-(R74-Pad2)
- R87 pad 1: /In16/T13 -> Net-(J21-Pad1)
- R87 pad 2: GND -> Net-(R87-Pad2)
- U10 pad 4: /In16/T13 -> Net-(J21-Pad1)
- U9 pad 4: /In16/T9 -> Net-(J17-Pad1)
