File: Opto_8/Opto_8.kicad_sch (KiCad schematic)
At the start: 75 parts, among them J1 Conn_01x06, J2 nmount SW Debug, J3 USB_C_Receptacle_USB2.0, J4 Conn_01x06, SW1 Reset, SW2 Boot, SW3 ADDRESS, U1 ADM3483, U14 LMV321, U2 W25Q128JVSIQ, U3 RP2040, U4 SN74AHCT1G125, U5 AP2112K-3.3, Y1 12MHz,18pF

Commit message: in16_drv8
Other:
- sheet Driver8 ports: added none; removed DRV_1, DRV_2, DRV_3, DRV_4, DRV_5, DRV_6, DRV_7, DRV_8
- title: IO_16x8_matrix -> Opto_8

Commit message: basic
Parts:
- renumbered C9 to C10, C10 to C11, C11 to C12, C12 to C13, C13 to C14, C14 to C15, C15 to C16, C16 to C17, C17 to C18, C18 to C19, C19 to C20, C20 to C21, C21 to C22, C22 to C23, C23 to C24, C24 to C25, C42 to C8, C8 to C9, D23 to D7, R12 to R10, R13 to R11, R14 to R12, R56 to R13, R57 to R14, R58 to R15, R15 to R16, R59 to R17, R60 to R18, R61 to R19, R62 to R20, R63 to R21, R64 to R22, R16 to R23, R17 to R24, R18 to R25, R19 to R26, R4 to R3, R6 to R4, R7 to R5, R8 to R6, R9 to R7, R10 to R8, R11 to R9, TP4 to TP1, TP5 to TP2, U14 to U3, U3 to U4, U4 to U5, U5 to U6
Connections:
- net Out_1: no longer names the net of U4.39 (GPIO27_ADC1)
- net Out_2: no longer names the net of U4.38 (GPIO26_ADC0)
- net Out_3: no longer names the net of U4.36 (GPIO24)
- net Out_4: no longer names the net of U4.35 (GPIO23)
- net Out_5: no longer names the net of U4.34 (GPIO22)
- net Out_6: no longer names the net of U4.32 (GPIO21)
- net Out_7: no longer names the net of U4.31 (GPIO20)
- net Out_8: no longer names the net of U4.30 (GPIO19)
Other:
- note added: "ADC/PWM?"
