File: Opto_8/rdi_sub_4x.kicad_sch (KiCad schematic)
At the start: 15 parts, among them U7 LM339

Commit message: basic
Parts:
- removed C28, C29: 100n, Capacitor_SMD:C_0402_1005Metric, symbol Device:C
- removed R39, R40, R45, R46: 10k, Resistor_SMD:R_0603_1608Metric, symbol Device:R
- removed R41, R43, R47, R49: 1k, Resistor_SMD:R_0603_1608Metric, symbol Device:R
- removed R42, R44, R48, R50: 2k, Resistor_SMD:R_0603_1608Metric, symbol Device:R
- removed U7: LM339, Package_SO:SOIC-14_3.9x8.7mm_P1.27mm, symbol Comparator:LM339
- added C32, C33: 100n, Capacitor_SMD:C_0402_1005Metric, symbol Device:C
- added J15, J16, J17, J18: Conn_01x02, Connector_Molex:Molex_KK-254_AE-6410-02A_1x02_P2.54mm_Vertical, symbol Connector_Generic:Conn_01x02
- added R63, R64, R67, R68: 10k, Resistor_SMD:R_0603_1608Metric, symbol Device:R
- added R65, R66, R69, R70: 1M, Resistor_SMD:R_0603_1608Metric, symbol Device:R
- added U9: LM339, Package_SO:SOIC-14_3.9x8.7mm_P1.27mm, symbol Comparator:LM339
Connections:
- net +3V3: now also R63.1, R64.1, R67.1, R68.1
- net +5V: now also C32.1, U9.3 (V+)
- net GND: now also C32.2, C33.2, J15.2 (Pin_2), J16.2 (Pin_2), J17.2 (Pin_2), J18.2 (Pin_2), R65.2, R66.2, R69.2, R70.2, U9.12 (V-)
- net RTN1_SUB: now also R63.2, U9.2
- net RTN2_SUB: now also R64.2, U9.1
- net RTN3_SUB: now also R67.2, U9.14
- net RTN4_SUB: now also R68.2, U9.13
- net TRM1_SUB: now also J15.1 (Pin_1), R65.1, U9.4 (-)
- net TRM2_SUB: now also J16.1 (Pin_1), R66.1, U9.6 (-)
- net TRM3_SUB: now also J17.1 (Pin_1), R69.1, U9.8 (-)
- net TRM4_SUB: now also J18.1 (Pin_1), R70.1, U9.10 (-)
- net V_SW_SUB: now also C33.1, U9.11 (+), U9.5 (+), U9.7 (+), U9.9 (+)

Commit message: configurable_inputs
Parts:
- removed R66, R69, R70: 1M, Resistor_SMD:R_0603_1608Metric, symbol Device:R
- added R73: 1k, Resistor_SMD:R_0603_1608Metric, symbol Device:R
- added R75, R77, R81, R83: 2k, Resistor_SMD:R_0603_1608Metric, symbol Device:R
- added R76, R80, R82: 1M, Resistor_SMD:R_0603_1608Metric, symbol Device:R
- renumbered J15 to J17, J16 to J18, J17 to J19, J18 to J20, R63 to R71, R64 to R72, R65 to R74, R67 to R78, R68 to R79
Connections:
- net GND: now also R75.2, R77.2, R81.2, R83.2; no longer J17.2 (Pin_2), J18.2 (Pin_2), J19.2 (Pin_2), J20.2 (Pin_2), R74.2
- net TRM1_SUB: now also R73.1; no longer J17.1 (Pin_1), R74.1, U9.4 (-)
- net TRM2_SUB: now also R76.1
- net TRM3_SUB: now also R80.1
- net TRM4_SUB: now also R82.1
- new net: J20.2 (Pin_2), R82.2, R83.1
- new net: J19.2 (Pin_2), R80.2, R81.1
- new net: J17.1 (Pin_1), R73.2, R74.1, U9.4 (-)
- new net: J17.2 (Pin_2), R74.2, R75.1
- new net: J18.2 (Pin_2), R76.2, R77.1
