File: Opto_16/In16.kicad_sch (KiCad schematic)
At the start: 9 parts, among them J15 Conn_01x10, J16 Conn_01x10

Commit message: V1.0.0
Parts:
- renumbered C26 to C34, C27 to C35, J15 to J16, J16 to J17, R43 to R51, R44 to R52, R45 to R53, R46 to R54
Other:
- title: Opto_8 -> Opto_16
Changed lines of the file:
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@@
   (paper "A4")
   (title_block
-    (title "Opto_8")
-    (date "2025-03-26")
-    (rev "0.1.0")
+    (title "Opto_16")
+    (date "2025-04-29")
+    (rev "1.0.0")
   )
   (junction (at 209.55 127) (diameter 0) (color 0 0 0 0)
@@
   (symbol (lib_id "Device:R") (at 209.55 132.08 0) (unit 1)
     (in_bom yes) (on_board yes) (fields_autoplaced)
-    (property "Reference" "R44" (id 0) (at 212.09 130.8099 0)
+    (property "Reference" "R52" (id 0) (at 212.09 130.8099 0)
       (effects (font (size 1.27 1.27)) (justify left))
     )
@@
   (symbol (lib_id "power:+5V") (at 200.66 33.02 0) (unit 1)
     (in_bom yes) (on_board yes)
-    (property "Reference" "#PWR072" (id 0) (at 200.66 36.83 0)
+    (property "Reference" "#PWR077" (id 0) (at 200.66 36.83 0)
       (effects (font (size 1.27 1.27)) hide)
     )
@@
   (symbol (lib_id "power:GND") (at 209.55 137.16 0) (unit 1)
     (in_bom yes) (on_board yes)
-    (property "Reference" "#PWR074" (id 0) (at 209.55 143.51 0)
+    (property "Reference" "#PWR079" (id 0) (at 209.55 143.51 0)
       (effects (font (size 1.27 1.27)) hide)
     )
@@
   (symbol (lib_id "power:+5V") (at 237.49 33.02 0) (unit 1)
     (in_bom yes) (on_board yes)
-    (property "Reference" "#PWR076" (id 0) (at 237.49 36.83 0)
+    (property "Reference" "#PWR081" (id 0) (at 237.49 36.83 0)
       (effects (font (size 1.27 1.27)) hide)
     )
@@
   (symbol (lib_id "Device:R") (at 247.65 121.92 0) (unit 1)
     (in_bom yes) (on_board yes) (fields_autoplaced)
-    (property "Reference" "R45" (id 0) (at 250.19 120.6499 0)
+    (property "Reference" "R53" (id 0) (at 250.19 120.6499 0)
       (effects (font (size 1.27 1.27)) (justify left))
     )
@@
   (symbol (lib_id "Device:C") (at 256.54 132.08 0) (unit 1)
     (in_bom yes) (on_board yes)
-    (property "Reference" "C27" (id 0) (at 259.08 130.81 0)
+    (property "Reference" "C35" (id 0) (at 259.08 130.81 0)
       (effects (font (size 1.27 1.27)) (justify left))
     )
@@
   (symbol (lib_id "Device:C") (at 218.44 132.08 0) (unit 1)
     (in_bom yes) (on_board yes)
-    (property "Reference" "C26" (id 0) (at 220.98 130.81 0)
+    (property "Reference" "C34" (id 0) (at 220.98 130.81 0)
       (effects (font (size 1.27 1.27)) (justify left))
     )
@@
   (symbol (lib_id "power:+5V") (at 247.65 116.84 0) (unit 1)
     (in_bom yes) (on_board yes)
-    (property "Reference" "#PWR077" (id 0) (at 247.65 120.65 0)
+    (property "Reference" "#PWR082" (id 0) (at 247.65 120.65 0)
       (effects (font (size 1.27 1.27)) hide)
     )
@@
   (symbol (lib_id "power:GND") (at 247.65 137.16 0) (unit 1)
     (in_bom yes) (on_board yes)
-    (property "Reference" "#PWR078" (id 0) (at 247.65 143.51 0)
+    (property "Reference" "#PWR083" (id 0) (at 247.65 143.51 0)
       (effects (font (size 1.27 1.27)) hide)
     )
@@
   (symbol (lib_id "power:GND") (at 218.44 137.16 0) (unit 1)
     (in_bom yes) (on_board yes)
-    (property "Reference" "#PWR075" (id 0) (at 218.44 143.51 0)
+    (property "Reference" "#PWR080" (id 0) (at 218.44 143.51 0)
       (effects (font (size 1.27 1.27)) hide)
     )
@@
   (symbol (lib_id "Connector_Generic:Conn_01x10") (at 246.38 45.72 0) (unit 1)
     (in_bom yes) (on_board yes) (fields_autoplaced)
-    (property "Reference" "J16" (id 0) (at 248.92 45.7199 0)
+    (property "Reference" "J17" (id 0) (at 248.92 45.7199 0)
       (effects (font (size 1.27 1.27)) (justify left))
     )
@@
   (symbol (lib_id "power:+5V") (at 209.55 116.84 0) (unit 1)
     (in_bom yes) (on_board yes)
-    (property "Reference" "#PWR073" (id 0) (at 209.55 120.65 0)
+    (property "Reference" "#PWR078" (id 0) (at 209.55 120.65 0)
       (effects (font (size 1.27 1.27)) hide)
     )
@@
   (symbol (lib_id "power:GND") (at 256.54 137.16 0) (unit 1)
     (in_bom yes) (on_board yes)
-    (property "Reference" "#PWR079" (id 0) (at 256.54 143.51 0)
+    (property "Reference" "#PWR084" (id 0) (at 256.54 143.51 0)
       (effects (font (size 1.27 1.27)) hide)
     )
@@
   (symbol (lib_id "Device:R") (at 209.55 121.92 0) (unit 1)
     (in_bom yes) (on_board yes) (fields_autoplaced)
-    (property "Reference" "R43" (id 0) (at 212.09 120.6499 0)
+    (property "Reference" "R51" (id 0) (at 212.09 120.6499 0)
       (effects (font (size 1.27 1.27)) (justify left))
     )
@@
   (symbol (lib_id "Device:R") (at 247.65 132.08 0) (unit 1)
     (in_bom yes) (on_board yes) (fields_autoplaced)
-    (property "Reference" "R46" (id 0) (at 250.19 130.8099 0)
+    (property "Reference" "R54" (id 0) (at 250.19 130.8099 0)
       (effects (font (size 1.27 1.27)) (justify left))
     )
@@
   (symbol (lib_id "Connector_Generic:Conn_01x10") (at 209.55 45.72 0) (unit 1)
     (in_bom yes) (on_board yes) (fields_autoplaced)
-    (property "Reference" "J15" (id 0) (at 212.09 45.7199 0)
-      (effects (font (size 1.27 1.27)) (justify left))
-    )
+    (property "Reference" "J16" (id 0) (at 212.09 45.7199 0)
+      (effects (font (size 1.27 1.27)) (justify left))
+    )
