File: Opto_16/Opto_16.kicad_pcb (KiCad board)
At the start: 2 copper layers, 99.7 x 67.3 mm, 189 parts, among them J1 Conn_01x06, J10 Conn_01x02, J11 Conn_01x02, J12 Conn_01x02, J13 Conn_01x02, J14 Conn_01x10, J15 Conn_01x10, J16 Conn_01x10, J17 Conn_01x02, J18 Conn_01x02, J19 Conn_01x02, J2 nmount SW Debug, J20 Conn_01x02, J21 Conn_01x02, J22 Conn_01x02, J23 Conn_01x02, J24 Conn_01x02, J3 USB_C_Receptacle_USB2.0, J4 Conn_01x06, J5 Conn_01x10, J6 Conn_01x02, J7 Conn_01x02, J8 Conn_01x02, J9 Conn_01x02, SW1 Reset, SW2 Boot, SW3 ADDRESS, U1 ADM3483, U10 LM339, U2 W25Q128JVSIQ, U3 LMV321, U4 RP2040, U5 SN74AHCT1G125, U6 AP2112K-3.3, U7 LM339, U8 LM339, U9 LM339, Y1 12MHz,18pF

Commit message: V1.0.0
Parts:
- added C20: 100n, Capacitor_SMD:C_0402_1005Metric, F.Cu at (168.5, 80.8)
- added C21: 100n, Capacitor_SMD:C_0402_1005Metric, F.Cu at (168.5, 78.4)
- added C23: 100n, Capacitor_SMD:C_0402_1005Metric, F.Cu at (167.3, 68.5)
- added C24: 100n, Capacitor_SMD:C_0402_1005Metric, F.Cu at (168.5, 75.7)
- added C25: 100n, Capacitor_SMD:C_0402_1005Metric, F.Cu at (168.5, 73.2)
- added C26: 100n, Capacitor_SMD:C_0402_1005Metric, F.Cu at (166.0, 68.4)
- added C27: 100n, Capacitor_SMD:C_0402_1005Metric, F.Cu at (168.5, 70.7)
- added C28: 100n, Capacitor_SMD:C_0402_1005Metric, F.Cu at (168.5, 68.5)
- added J4: Conn_01x10, Connector_PinSocket_2.54mm:PinSocket_1x10_P2.54mm_Vertical, F.Cu at (172.3, 82.9)
- added R21: 1k, Resistor_SMD:R_0402_1005Metric, F.Cu at (169.8, 80.8)
- added R22: 1k, Resistor_SMD:R_0402_1005Metric, F.Cu at (169.8, 78.4)
- added R23: 1k, Resistor_SMD:R_0402_1005Metric, F.Cu at (169.8, 75.7)
- added R24: 1k, Resistor_SMD:R_0402_1005Metric, F.Cu at (169.8, 73.2)
- added R25: 1k, Resistor_SMD:R_0402_1005Metric, F.Cu at (169.8, 70.7)
- added R26: 1k, Resistor_SMD:R_0402_1005Metric, F.Cu at (169.8, 68.2)
- added R29: 1k, Resistor_SMD:R_0402_1005Metric, F.Cu at (169.8, 65.7)
- added R30: 1k, Resistor_SMD:R_0402_1005Metric, F.Cu at (169.8, 63.4)
- moved J17 45.0 mm to (135.4, 105.4)
- moved R88 42.4 mm to (126.0, 87.8), turned to -90 degrees
- moved J16 41.9 mm to (180.8, 105.4)
- moved R79 38.9 mm to (126.0, 78.6), turned to -90 degrees
- moved R87 38.0 mm to (126.0, 84.7), turned to -90 degrees
- moved R99 37.9 mm to (108.5, 85.5), turned to 90 degrees
- moved R98 37.4 mm to (109.2, 87.7), turned to 180 degrees
- moved R95 34.9 mm to (126.8, 90.4), turned to 180 degrees
- moved J8 34.2 mm to (195.2, 66.9)
- moved J13 34.1 mm to (195.2, 98.0)
- moved R80 34.0 mm to (126.0, 81.7), turned to 90 degrees
- moved C42 32.6 mm to (122.1, 89.4)
- moved C40 31.1 mm to (122.1, 79.4)
- moved R102 31.0 mm to (108.5, 91.5), turned to 90 degrees
- moved R101 30.8 mm to (108.5, 94.5), turned to 90 degrees
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- renumbered C20 to C22, C21 to C29, C22 to C30, C23 to C31, C24 to C32, C25 to C33, C26 to C34, C27 to C35, C28 to C36, C29 to C37, C30 to C38, C31 to C39, C32 to C40, C33 to C41, C34 to C42, C35 to C43, J9 to J10, J10 to J11, J11 to J12, J12 to J13, J13 to J14, J14 to J15, J15 to J16, J16 to J17, J17 to J18, J18 to J19, J19 to J20, J20 to J21, J21 to J22, J22 to J23, J23 to J24, J24 to J25, J4 to J5, J5 to J6, J6 to J7, J7 to J8, J8 to J9, R92 to R100, R93 to R101, R94 to R102, R95 to R103, R96 to R104, R97 to R105, R98 to R106, R99 to R107, R100 to R108, R101 to R109, R102 to R110, R21 to R27, R22 to R28, R23 to R31, R24 to R32, R25 to R33, R26 to R34, R27 to R35, R28 to R36, R29 to R37, R30 to R38, R31 to R39, R32 to R40, R33 to R41, R34 to R42, R35 to R43, R36 to R44, R37 to R45, R38 to R46, R39 to R47, R40 to R48, R41 to R49, R42 to R50, R43 to R51, R44 to R52, R45 to R53, R46 to R54, R47 to R55, R48 to R56, R49 to R57, R50 to R58, R51 to R59, R52 to R60, R53 to R61, R54 to R62, R55 to R63, R56 to R64, R57 to R65, R58 to R66, R59 to R67, R60 to R68, R61 to R69, R62 to R70, R63 to R71, R64 to R72, R65 to R73, R66 to R74, R67 to R75, R68 to R76, R69 to R77, R70 to R78, R71 to R79, R72 to R80, R73 to R81, R74 to R82, R75 to R83, R76 to R84, R77 to R85, R78 to R86, R79 to R87, R80 to R88, R81 to R89, R82 to R90, R83 to R91, R84 to R92, R85 to R93, R86 to R94, R87 to R95, R88 to R96, R89 to R97, R90 to R98, R91 to R99
Connections:
- U4 pad 30: unconnected-(U4-Pad30) -> Net-(R21-Pad1)
- U4 pad 31: unconnected-(U4-Pad31) -> Net-(R22-Pad1)
- U4 pad 32: unconnected-(U4-Pad32) -> Net-(R23-Pad1)
- U4 pad 34: unconnected-(U4-Pad34) -> Net-(R24-Pad1)
- U4 pad 35: unconnected-(U4-Pad35) -> Net-(R25-Pad1)
- U4 pad 36: unconnected-(U4-Pad36) -> Net-(R26-Pad1)
- U4 pad 38: unconnected-(U4-Pad38) -> Net-(C23-Pad1)
- U4 pad 39: unconnected-(U4-Pad39) -> Net-(C26-Pad1)
Routing:
- net Net-(J24-Pad2): track 181.7 -> 5.76 mm, vias 2 -> 0
- net +5V: track 387.7 -> 240.7 mm, vias 27 -> 8
- net /In16/T14: track 144.2 -> 15.5 mm
- net GND: track 473.8 -> 345.3 mm, vias 385 -> 371
- net /In16/T5: track 22.0 -> 144.5 mm
- net /In16/T8: track 14.2 -> 130.3 mm
- net /In16/T7: track 17.2 -> 130.9 mm
- net /In16/T6: track 22.5 -> 134.4 mm
- net /In16/T3: track 56.6 -> 138.3 mm
- net /In16/T4: track 54.1 -> 135.3 mm
- net /In16/T1: track 64.7 -> 142.4 mm
- net /In16/T13: track 81.0 -> 20.7 mm, vias 0 -> 1
- net /In16/T2: track 76.8 -> 134.1 mm
- net /Driver8/D8: track 6.07 -> 58.6 mm
- net unconnected-(U4-Pad36): track 44.8 -> 0.00 mm, vias 2 -> 0
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Other:
- board text added: "26"
- board text added: "27"
- board text added: "28"
- board text added: "29"
- board text added: "30"
- board text added: "31"
- board text added: "32"
- board text added: "5V"
- board text added: "A0"
- board text added: "A1"
- board text added: "Opto_16"
- board text added: "P19"
- board text added: "P20"
- board text added: "P21"
- board text added: "P22"
- board text added: "P23"
- board text added: "P24"
- board text removed: "IO_16x8_matrix"
