File: Opto_16/Opto_16.kicad_sch (KiCad schematic)
At the start: 75 parts, among them J1 Conn_01x06, J2 nmount SW Debug, J3 USB_C_Receptacle_USB2.0, J4 Conn_01x06, SW1 Reset, SW2 Boot, SW3 ADDRESS, U1 ADM3483, U2 W25Q128JVSIQ, U3 LMV321, U4 RP2040, U5 SN74AHCT1G125, U6 AP2112K-3.3, Y1 12MHz,18pF

Commit message: V1.0.0
Parts:
- added C20, C21, C23, C24, C25, C26, C27, C28: 100n, Capacitor_SMD:C_0402_1005Metric, symbol Device:C
- added J4: Conn_01x10, Connector_PinSocket_2.54mm:PinSocket_1x10_P2.54mm_Vertical, symbol Connector_Generic:Conn_01x10
- added R21, R22, R23, R24, R25, R26, R29, R30: 1k, Resistor_SMD:R_0402_1005Metric, symbol Device:R
- renumbered C20 to C22, C21 to C29, C22 to C30, C23 to C31, C24 to C32, C25 to C33, J4 to J5, R21 to R27, R22 to R28, R23 to R31, R24 to R32, R25 to R33, R26 to R34
Connections:
- net GND: now also C20.1, C21.1, C23.2, C24.1, C25.1, C26.2, C27.1, C28.1, J4.1 (Pin_1), J4.10 (Pin_10)
- net at U4.30 (GPIO19): now also R21.1
- net at U4.31 (GPIO20): now also R22.1
- net at U4.32 (GPIO21): now also R23.1
- net at U4.34 (GPIO22): now also R24.1
- net at U4.35 (GPIO23): now also R25.1
- net at U4.36 (GPIO24): now also R26.1
- net at U4.38 (GPIO26_ADC0): now also C23.1, R29.1
- net at U4.39 (GPIO27_ADC1): now also C26.1, R30.1
- new net: C20.2, J4.2 (Pin_2), R21.2
- new net: C21.2, J4.3 (Pin_3), R22.2
- new net: C24.2, J4.4 (Pin_4), R23.2
- new net: C25.2, J4.5 (Pin_5), R24.2
- new net: C27.2, J4.6 (Pin_6), R25.2
- new net: C28.2, J4.7 (Pin_7), R26.2
- new net ADC0: J4.8 (Pin_8), R29.2
- new net ADC1: J4.9 (Pin_9), R30.2
Other:
- note removed: "ADC/PWM?"
- title: Opto_8 -> Opto_16
