File: Opto_16/rdi_sub_4x.kicad_sch (KiCad schematic)
At the start: 23 parts, among them J17 Conn_01x02, J18 Conn_01x02, J19 Conn_01x02, J20 Conn_01x02, U9 LM339

Commit message: V1.0.0
Parts:
- renumbered C32 to C40, C33 to C41, J17 to J18, J18 to J19, J19 to J20, J20 to J21, R71 to R79, R72 to R80, R73 to R81, R74 to R82, R75 to R83, R76 to R84, R77 to R85, R78 to R86, R79 to R87, R80 to R88, R81 to R89, R82 to R90, R83 to R91, R84 to R92, R85 to R93, R86 to R94
Other:
- title: Opto_8 -> Opto_16
Changed lines of the file:
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@@
   (paper "A4")
   (title_block
-    (title "Opto_8")
-    (date "2025-03-26")
-    (rev "0.1.0")
+    (title "Opto_16")
+    (date "2025-04-29")
+    (rev "1.0.0")
   )
   (junction (at 175.26 102.87) (diameter 0) (color 0 0 0 0)
@@
   (symbol (lib_id "Device:R") (at 175.26 96.52 0) (unit 1)
     (in_bom yes) (on_board yes)
-    (property "Reference" "R80" (id 0) (at 175.26 97.79 90)
+    (property "Reference" "R88" (id 0) (at 175.26 97.79 90)
       (effects (font (size 1.27 1.27)) (justify left))
     )
@@
   (symbol (lib_id "power:+3V3") (at 175.26 91.44 0) (unit 1)
     (in_bom yes) (on_board yes)
-    (property "Reference" "#PWR0110" (id 0) (at 175.26 95.25 0)
+    (property "Reference" "#PWR0115" (id 0) (at 175.26 95.25 0)
       (effects (font (size 1.27 1.27)) hide)
     )
@@
   (symbol (lib_id "Device:R") (at 208.28 105.41 0) (unit 1)
     (in_bom yes) (on_board yes) (fields_autoplaced)
-    (property "Reference" "R85" (id 0) (at 210.82 104.1399 0)
+    (property "Reference" "R93" (id 0) (at 210.82 104.1399 0)
       (effects (font (size 1.27 1.27)) (justify left))
     )
@@
   (symbol (lib_id "power:GND") (at 104.14 71.12 0) (unit 1)
     (in_bom yes) (on_board yes)
-    (property "Reference" "#PWR0106" (id 0) (at 104.14 77.47 0)
+    (property "Reference" "#PWR0111" (id 0) (at 104.14 77.47 0)
       (effects (font (size 1.27 1.27)) hide)
     )
@@
   (symbol (lib_id "Device:C") (at 72.39 163.83 0) (unit 1)
     (in_bom yes) (on_board yes)
-    (property "Reference" "C32" (id 0) (at 71.12 162.56 90)
+    (property "Reference" "C40" (id 0) (at 71.12 162.56 90)
       (effects (font (size 1.27 1.27)) (justify left))
     )
@@
   (symbol (lib_id "Device:R") (at 208.28 66.04 0) (unit 1)
     (in_bom yes) (on_board yes) (fields_autoplaced)
-    (property "Reference" "R83" (id 0) (at 210.82 64.7699 0)
+    (property "Reference" "R91" (id 0) (at 210.82 64.7699 0)
       (effects (font (size 1.27 1.27)) (justify left))
     )
@@
   (symbol (lib_id "Device:R") (at 208.28 55.88 0) (unit 1)
     (in_bom yes) (on_board yes) (fields_autoplaced)
-    (property "Reference" "R82" (id 0) (at 210.82 54.6099 0)
+    (property "Reference" "R90" (id 0) (at 210.82 54.6099 0)
       (effects (font (size 1.27 1.27)) (justify left))
     )
@@
   (symbol (lib_id "power:GND") (at 208.28 71.12 0) (unit 1)
     (in_bom yes) (on_board yes)
-    (property "Reference" "#PWR0111" (id 0) (at 208.28 77.47 0)
+    (property "Reference" "#PWR0116" (id 0) (at 208.28 77.47 0)
       (effects (font (size 1.27 1.27)) hide)
     )
@@
   (symbol (lib_id "Connector_Generic:Conn_01x02") (at 220.98 50.8 0) (unit 1)
     (in_bom yes) (on_board yes) (fields_autoplaced)
-    (property "Reference" "J19" (id 0) (at 223.52 50.7999 0)
+    (property "Reference" "J20" (id 0) (at 223.52 50.7999 0)
       (effects (font (size 1.27 1.27)) (justify left))
     )
@@
   (symbol (lib_id "Connector_Generic:Conn_01x02") (at 220.98 100.33 0) (unit 1)
     (in_bom yes) (on_board yes) (fields_autoplaced)
-    (property "Reference" "J20" (id 0) (at 223.52 100.3299 0)
+    (property "Reference" "J21" (id 0) (at 223.52 100.3299 0)
       (effects (font (size 1.27 1.27)) (justify left))
     )
@@
   (symbol (lib_id "Device:R") (at 104.14 55.88 0) (unit 1)
     (in_bom yes) (on_board yes) (fields_autoplaced)
-    (property "Reference" "R74" (id 0) (at 106.68 54.6099 0)
+    (property "Reference" "R82" (id 0) (at 106.68 54.6099 0)
       (effects (font (size 1.27 1.27)) (justify left))
     )
@@
   (symbol (lib_id "power:+3V3") (at 71.12 41.91 0) (unit 1)
     (in_bom yes) (on_board yes)
-    (property "Reference" "#PWR0102" (id 0) (at 71.12 45.72 0)
+    (property "Reference" "#PWR0107" (id 0) (at 71.12 45.72 0)
       (effects (font (size 1.27 1.27)) hide)
     )
@@
   (symbol (lib_id "power:GND") (at 81.28 172.72 0) (unit 1)
     (in_bom yes) (on_board yes)
-    (property "Reference" "#PWR0105" (id 0) (at 81.28 179.07 0)
+    (property "Reference" "#PWR0110" (id 0) (at 81.28 179.07 0)
       (effects (font (size 1.27 1.27)) hide)
     )
@@
   (symbol (lib_id "Device:R") (at 175.26 46.99 0) (unit 1)
     (in_bom yes) (on_board yes)
-    (property "Reference" "R79" (id 0) (at 175.26 48.26 90)
+    (property "Reference" "R87" (id 0) (at 175.26 48.26 90)
       (effects (font (size 1.27 1.27)) (justify left))
     )
@@
   (symbol (lib_id "Device:R") (at 208.28 44.45 0) (unit 1)
     (in_bom yes) (on_board yes) (fields_autoplaced)
-    (property "Reference" "R81" (id 0) (at 210.82 43.1799 0)
+    (property "Reference" "R89" (id 0) (at 210.82 43.1799 0)
       (effects (font (size 1.27 1.27)) (justify left))
     )
@@
   (symbol (lib_id "power:GND") (at 104.14 120.65 0) (unit 1)
     (in_bom yes) (on_board yes)
-    (property "Reference" "#PWR0107" (id 0) (at 104.14 127 0)
+    (property "Reference" "#PWR0112" (id 0) (at 104.14 127 0)
       (effects (font (size 1.27 1.27)) hide)
     )
@@
   (symbol (lib_id "Device:R") (at 104.14 66.04 0) (unit 1)
     (in_bom yes) (on_board yes) (fields_autoplaced)
-    (property "Reference" "R75" (id 0) (at 106.68 64.7699 0)
+    (property "Reference" "R83" (id 0) (at 106.68 64.7699 0)
       (effects (font (size 1.27 1.27)) (justify left))
     )
@@
   (symbol (lib_id "Device:R") (at 208.28 115.57 0) (unit 1)
     (in_bom yes) (on_board yes) (fields_autoplaced)
-    (property "Reference" "R86" (id 0) (at 210.82 114.2999 0)
+    (property "Reference" "R94" (id 0) (at 210.82 114.2999 0)
       (effects (font (size 1.27 1.27)) (justify left))
     )
@@
   (symbol (lib_id "Device:R") (at 71.12 96.52 0) (unit 1)
     (in_bom yes) (on_board yes)
-    (property "Reference" "R72" (id 0) (at 71.12 97.79 90)
+    (property "Reference" "R80" (id 0) (at 71.12 97.79 90)
       (effects (font (size 1.27 1.27)) (justify left))
     )
@@
   (symbol (lib_id "Device:R") (at 104.14 105.41 0) (unit 1)
     (in_bom yes) (on_board yes) (fields_autoplaced)
-    (property "Reference" "R77" (id 0) (at 106.68 104.1399 0)
+    (property "Reference" "R85" (id 0) (at 106.68 104.1399 0)
       (effects (font (size 1.27 1.27)) (justify left))
     )
@@
   (symbol (lib_id "Connector_Generic:Conn_01x02") (at 116.84 100.33 0) (unit 1)
     (in_bom yes) (on_board yes) (fields_autoplaced)
-    (property "Reference" "J18" (id 0) (at 119.38 100.3299 0)
+    (property "Reference" "J19" (id 0) (at 119.38 100.3299 0)
       (effects (font (size 1.27 1.27)) (justify left))
     )
@@
   (symbol (lib_id "Device:R") (at 104.14 115.57 0) (unit 1)
     (in_bom yes) (on_board yes) (fields_autoplaced)
-    (property "Reference" "R78" (id 0) (at 106.68 114.2999 0)
+    (property "Reference" "R86" (id 0) (at 106.68 114.2999 0)
       (effects (font (size 1.27 1.27)) (justify left))
     )
@@
   (symbol (lib_id "Device:R") (at 104.14 44.45 0) (unit 1)
     (in_bom yes) (on_board yes) (fields_autoplaced)
-    (property "Reference" "R73" (id 0) (at 106.68 43.1799 0)
+    (property "Reference" "R81" (id 0) (at 106.68 43.1799 0)
       (effects (font (size 1.27 1.27)) (justify left))
     )
@@
   (symbol (lib_id "power:+3V3") (at 175.26 41.91 0) (unit 1)
     (in_bom yes) (on_board yes)
-    (property "Reference" "#PWR0109" (id 0) (at 175.26 45.72 0)
+    (property "Reference" "#PWR0114" (id 0) (at 175.26 45.72 0)
       (effects (font (size 1.27 1.27)) hide)
     )
@@
   (symbol (lib_id "power:+3V3") (at 71.12 91.44 0) (unit 1)
     (in_bom yes) (on_board yes)
-    (property "Reference" "#PWR0103" (id 0) (at 71.12 95.25 0)
+    (property "Reference" "#PWR0108" (id 0) (at 71.12 95.25 0)
       (effects (font (size 1.27 1.27)) hide)
     )
@@
   (symbol (lib_id "power:+5V") (at 81.28 152.4 0) (unit 1)
     (in_bom yes) (on_board yes)
-    (property "Reference" "#PWR0104" (id 0) (at 81.28 156.21 0)
+    (property "Reference" "#PWR0109" (id 0) (at 81.28 156.21 0)
       (effects (font (size 1.27 1.27)) hide)
     )
@@
   (symbol (lib_id "Device:C") (at 110.49 163.83 0) (unit 1)
     (in_bom yes) (on_board yes)
-    (property "Reference" "C33" (id 0) (at 109.22 162.56 90)
+    (property "Reference" "C41" (id 0) (at 109.22 162.56 90)
       (effects (font (size 1.27 1.27)) (justify left))
     )
@@
   (symbol (lib_id "Connector_Generic:Conn_01x02") (at 116.84 50.8 0) (unit 1)
     (in_bom yes) (on_board yes) (fields_autoplaced)
-    (property "Reference" "J17" (id 0) (at 119.38 50.7999 0)
+    (property "Reference" "J18" (id 0) (at 119.38 50.7999 0)
       (effects (font (size 1.27 1.27)) (justify left))
     )
@@
   (symbol (lib_id "power:GND") (at 208.28 120.65 0) (unit 1)
     (in_bom yes) (on_board yes)
-    (property "Reference" "#PWR0112" (id 0) (at 208.28 127 0)
+    (property "Reference" "#PWR0117" (id 0) (at 208.28 127 0)
       (effects (font (size 1.27 1.27)) hide)
     )
@@
   (symbol (lib_id "power:GND") (at 110.49 172.72 0) (unit 1)
     (in_bom yes) (on_board yes)
-    (property "Reference" "#PWR0108" (id 0) (at 110.49 179.07 0)
+    (property "Reference" "#PWR0113" (id 0) (at 110.49 179.07 0)
       (effects (font (size 1.27 1.27)) hide)
     )
@@
   (symbol (lib_id "Device:R") (at 71.12 46.99 0) (unit 1)
     (in_bom yes) (on_board yes)
-    (property "Reference" "R71" (id 0) (at 71.12 48.26 90)
+    (property "Reference" "R79" (id 0) (at 71.12 48.26 90)
       (effects (font (size 1.27 1.27)) (justify left))
     )
@@
   (symbol (lib_id "Device:R") (at 208.28 93.98 0) (unit 1)
     (in_bom yes) (on_board yes) (fields_autoplaced)
-    (property "Reference" "R84" (id 0) (at 210.82 92.7099 0)
+    (property "Reference" "R92" (id 0) (at 210.82 92.7099 0)
       (effects (font (size 1.27 1.27)) (justify left))
     )
@@
   (symbol (lib_id "Device:R") (at 104.14 93.98 0) (unit 1)
     (in_bom yes) (on_board yes) (fields_autoplaced)
-    (property "Reference" "R76" (id 0) (at 106.68 92.7099 0)
-      (effects (font (size 1.27 1.27)) (justify left))
-    )
+    (property "Reference" "R84" (id 0) (at 106.68 92.7099 0)
+      (effects (font (size 1.27 1.27)) (justify left))
+    )
