File: Opto_16/rtn_sub_4x.kicad_sch (KiCad schematic)
At the start: 15 parts, among them U7 LM339

Commit message: V1.0.0
Parts:
- renumbered C28 to C36, C29 to C37, R47 to R55, R48 to R56, R49 to R57, R50 to R58, R51 to R59, R52 to R60, R53 to R61, R54 to R62, R55 to R63, R56 to R64, R57 to R65, R58 to R66
Other:
- title: Opto_8 -> Opto_16
Changed lines of the file:
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@@
   (paper "A4")
   (title_block
-    (title "Opto_8")
-    (date "2025-03-26")
-    (rev "0.1.0")
+    (title "Opto_16")
+    (date "2025-04-29")
+    (rev "1.0.0")
   )
   (junction (at 175.26 102.87) (diameter 0) (color 0 0 0 0)
@@
   (symbol (lib_id "Device:R") (at 71.12 96.52 0) (unit 1)
     (in_bom yes) (on_board yes)
-    (property "Reference" "R48" (id 0) (at 71.12 97.79 90)
+    (property "Reference" "R56" (id 0) (at 71.12 97.79 90)
       (effects (font (size 1.27 1.27)) (justify left))
     )
@@
   (symbol (lib_id "power:GND") (at 104.14 62.23 0) (unit 1)
     (in_bom yes) (on_board yes)
-    (property "Reference" "#PWR084" (id 0) (at 104.14 68.58 0)
+    (property "Reference" "#PWR089" (id 0) (at 104.14 68.58 0)
       (effects (font (size 1.27 1.27)) hide)
     )
@@
   (symbol (lib_id "power:GND") (at 81.28 172.72 0) (unit 1)
     (in_bom yes) (on_board yes)
-    (property "Reference" "#PWR083" (id 0) (at 81.28 179.07 0)
+    (property "Reference" "#PWR088" (id 0) (at 81.28 179.07 0)
       (effects (font (size 1.27 1.27)) hide)
     )
@@
   (symbol (lib_id "Device:C") (at 110.49 163.83 0) (unit 1)
     (in_bom yes) (on_board yes)
-    (property "Reference" "C29" (id 0) (at 109.22 162.56 90)
+    (property "Reference" "C37" (id 0) (at 109.22 162.56 90)
       (effects (font (size 1.27 1.27)) (justify left))
     )
@@
   (symbol (lib_id "power:+3V3") (at 71.12 91.44 0) (unit 1)
     (in_bom yes) (on_board yes)
-    (property "Reference" "#PWR081" (id 0) (at 71.12 95.25 0)
+    (property "Reference" "#PWR086" (id 0) (at 71.12 95.25 0)
       (effects (font (size 1.27 1.27)) hide)
     )
@@
   (symbol (lib_id "power:GND") (at 208.28 62.23 0) (unit 1)
     (in_bom yes) (on_board yes)
-    (property "Reference" "#PWR089" (id 0) (at 208.28 68.58 0)
+    (property "Reference" "#PWR094" (id 0) (at 208.28 68.58 0)
       (effects (font (size 1.27 1.27)) hide)
     )
@@
   (symbol (lib_id "Device:C") (at 72.39 163.83 0) (unit 1)
     (in_bom yes) (on_board yes)
-    (property "Reference" "C28" (id 0) (at 71.12 162.56 90)
+    (property "Reference" "C36" (id 0) (at 71.12 162.56 90)
       (effects (font (size 1.27 1.27)) (justify left))
     )
@@
   (symbol (lib_id "Device:R") (at 104.14 46.99 0) (unit 1)
     (in_bom yes) (on_board yes) (fields_autoplaced)
-    (property "Reference" "R49" (id 0) (at 106.68 45.7199 0)
+    (property "Reference" "R57" (id 0) (at 106.68 45.7199 0)
       (effects (font (size 1.27 1.27)) (justify left))
     )
@@
   (symbol (lib_id "power:+3V3") (at 71.12 41.91 0) (unit 1)
     (in_bom yes) (on_board yes)
-    (property "Reference" "#PWR080" (id 0) (at 71.12 45.72 0)
+    (property "Reference" "#PWR085" (id 0) (at 71.12 45.72 0)
       (effects (font (size 1.27 1.27)) hide)
     )
@@
   (symbol (lib_id "Device:R") (at 175.26 46.99 0) (unit 1)
     (in_bom yes) (on_board yes)
-    (property "Reference" "R53" (id 0) (at 175.26 48.26 90)
+    (property "Reference" "R61" (id 0) (at 175.26 48.26 90)
       (effects (font (size 1.27 1.27)) (justify left))
     )
@@
   (symbol (lib_id "Device:R") (at 208.28 106.68 0) (unit 1)
     (in_bom yes) (on_board yes) (fields_autoplaced)
-    (property "Reference" "R58" (id 0) (at 210.82 105.4099 0)
+    (property "Reference" "R66" (id 0) (at 210.82 105.4099 0)
       (effects (font (size 1.27 1.27)) (justify left))
     )
@@
   (symbol (lib_id "power:GND") (at 110.49 172.72 0) (unit 1)
     (in_bom yes) (on_board yes)
-    (property "Reference" "#PWR086" (id 0) (at 110.49 179.07 0)
+    (property "Reference" "#PWR091" (id 0) (at 110.49 179.07 0)
       (effects (font (size 1.27 1.27)) hide)
     )
@@
   (symbol (lib_id "power:+3V3") (at 175.26 91.44 0) (unit 1)
     (in_bom yes) (on_board yes)
-    (property "Reference" "#PWR088" (id 0) (at 175.26 95.25 0)
+    (property "Reference" "#PWR093" (id 0) (at 175.26 95.25 0)
       (effects (font (size 1.27 1.27)) hide)
     )
@@
   (symbol (lib_id "Device:R") (at 208.28 96.52 0) (unit 1)
     (in_bom yes) (on_board yes) (fields_autoplaced)
-    (property "Reference" "R57" (id 0) (at 210.82 95.2499 0)
+    (property "Reference" "R65" (id 0) (at 210.82 95.2499 0)
       (effects (font (size 1.27 1.27)) (justify left))
     )
@@
   (symbol (lib_id "Device:R") (at 208.28 57.15 0) (unit 1)
     (in_bom yes) (on_board yes) (fields_autoplaced)
-    (property "Reference" "R56" (id 0) (at 210.82 55.8799 0)
+    (property "Reference" "R64" (id 0) (at 210.82 55.8799 0)
       (effects (font (size 1.27 1.27)) (justify left))
     )
@@
   (symbol (lib_id "power:GND") (at 104.14 111.76 0) (unit 1)
     (in_bom yes) (on_board yes)
-    (property "Reference" "#PWR085" (id 0) (at 104.14 118.11 0)
+    (property "Reference" "#PWR090" (id 0) (at 104.14 118.11 0)
       (effects (font (size 1.27 1.27)) hide)
     )
@@
   (symbol (lib_id "Device:R") (at 71.12 46.99 0) (unit 1)
     (in_bom yes) (on_board yes)
-    (property "Reference" "R47" (id 0) (at 71.12 48.26 90)
+    (property "Reference" "R55" (id 0) (at 71.12 48.26 90)
       (effects (font (size 1.27 1.27)) (justify left))
     )
@@
   (symbol (lib_id "Device:R") (at 104.14 106.68 0) (unit 1)
     (in_bom yes) (on_board yes) (fields_autoplaced)
-    (property "Reference" "R52" (id 0) (at 106.68 105.4099 0)
+    (property "Reference" "R60" (id 0) (at 106.68 105.4099 0)
       (effects (font (size 1.27 1.27)) (justify left))
     )
@@
   (symbol (lib_id "power:+3V3") (at 175.26 41.91 0) (unit 1)
     (in_bom yes) (on_board yes)
-    (property "Reference" "#PWR087" (id 0) (at 175.26 45.72 0)
+    (property "Reference" "#PWR092" (id 0) (at 175.26 45.72 0)
       (effects (font (size 1.27 1.27)) hide)
     )
@@
   (symbol (lib_id "Device:R") (at 104.14 57.15 0) (unit 1)
     (in_bom yes) (on_board yes) (fields_autoplaced)
-    (property "Reference" "R50" (id 0) (at 106.68 55.8799 0)
+    (property "Reference" "R58" (id 0) (at 106.68 55.8799 0)
       (effects (font (size 1.27 1.27)) (justify left))
     )
@@
   (symbol (lib_id "Device:R") (at 104.14 96.52 0) (unit 1)
     (in_bom yes) (on_board yes) (fields_autoplaced)
-    (property "Reference" "R51" (id 0) (at 106.68 95.2499 0)
+    (property "Reference" "R59" (id 0) (at 106.68 95.2499 0)
       (effects (font (size 1.27 1.27)) (justify left))
     )
@@
   (symbol (lib_id "Device:R") (at 208.28 46.99 0) (unit 1)
     (in_bom yes) (on_board yes) (fields_autoplaced)
-    (property "Reference" "R55" (id 0) (at 210.82 45.7199 0)
+    (property "Reference" "R63" (id 0) (at 210.82 45.7199 0)
       (effects (font (size 1.27 1.27)) (justify left))
     )
@@
   (symbol (lib_id "Device:R") (at 175.26 96.52 0) (unit 1)
     (in_bom yes) (on_board yes)
-    (property "Reference" "R54" (id 0) (at 175.26 97.79 90)
+    (property "Reference" "R62" (id 0) (at 175.26 97.79 90)
       (effects (font (size 1.27 1.27)) (justify left))
     )
@@
   (symbol (lib_id "power:+5V") (at 81.28 152.4 0) (unit 1)
     (in_bom yes) (on_board yes)
-    (property "Reference" "#PWR082" (id 0) (at 81.28 156.21 0)
+    (property "Reference" "#PWR087" (id 0) (at 81.28 156.21 0)
       (effects (font (size 1.27 1.27)) hide)
     )
@@
   (symbol (lib_id "power:GND") (at 208.28 111.76 0) (unit 1)
     (in_bom yes) (on_board yes)
-    (property "Reference" "#PWR090" (id 0) (at 208.28 118.11 0)
-      (effects (font (size 1.27 1.27)) hide)
-    )
+    (property "Reference" "#PWR095" (id 0) (at 208.28 118.11 0)
+      (effects (font (size 1.27 1.27)) hide)
+    )
